File: hardware/SmartScale2-PCB.kicad_sch (KiCad schematic)
At the start: 57 parts, among them J1 Conn_ARM_JTAG_SWD_10, J2 USB_C_Receptacle_USB2.0_16P, J3 Conn_01x02, J4 Conn_01x04, J5 Conn_01x03_MountingPin, J6 Conn_01x04_MountingPin, Q1 MMBT4403, SW1 SW_Push_JTP-1130, U1 ESP32-C6-WROOM-1, U2 MCP73831-2-OT, U3 HX711, U4 AP63203WU, U5 USBLC6-2SC6, U6 TTP223-BA6

Commit message: Update for the 4MB variant
Parts:
- U1: value ESP32-C6-WROOM-1 -> ESP32-C6-WROOM-1-N4
Changed lines of the file:
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@@
 			)
 		)
-		(property "Value" "ESP32-C6-WROOM-1"
+		(property "Value" "ESP32-C6-WROOM-1-N4"
 			(at 64.3733 27.94 0)
 			(show_name no)
